File: hw/Mechaduino-multi/Mechaduino-planzero.kicad_sch (KiCad schematic)
At the start: 22 parts, among them IC1 A4954ELPTR-T, J1 Conn_01x05, J2 SPI, J3 SPI_PWR, U1 ATtiny24-20MU, U2 AS5047D

Commit message: updates
Parts:
- added C10, C9: (no value), symbol Device:C
- added J4: (no value), symbol Connector_Generic:Conn_01x04
- added U3: (no value), symbol Regulator_Linear:TLV70033_SOT353
Connections:
- net +3V3: now also C10.1, U3.5 (OUT); no longer J1.5 (Pin_5)
- net PAS1: now also J4.4 (Pin_4)
- net PAS2: now also J4.3 (Pin_3)
- net PAS3: now also J4.2 (Pin_2)
- net PAS4: now also J4.1 (Pin_1)
- net VCC: now also C9.1, U3.1 (IN), U3.3 (EN)
- new net: C10.2, C9.2, U3.2 (GND)
