File: hw/Mechaduino-multi/Mechaduino-planzero.kicad_pcb (KiCad board)
At the start: 2 copper layers, 42.2 x 42.2 mm, 4 parts

Commit message: Some updates
Parts:
- added C1: 100n, Capacitor_SMD:C_0805_2012Metric_Pad1.18x1.45mm_HandSolder, F.Cu at (113.0, 109.0)
- added C10: 1uF, Capacitor_SMD:C_0805_2012Metric_Pad1.18x1.45mm_HandSolder, F.Cu at (141.9, 110.7)
- added C2: 4.7u, Capacitor_SMD:C_0805_2012Metric_Pad1.18x1.45mm_HandSolder, F.Cu at (137.9, 116.7)
- added C3: 100n, Capacitor_SMD:C_0805_2012Metric_Pad1.18x1.45mm_HandSolder, F.Cu at (117.8, 114.3)
- added C4: 100n, Capacitor_SMD:C_0805_2012Metric_Pad1.18x1.45mm_HandSolder, F.Cu at (121.6, 114.3)
- added C5: 100n, Capacitor_SMD:C_0805_2012Metric_Pad1.18x1.45mm_HandSolder, F.Cu at (131.3, 118.7)
- added C6: 100uF, Capacitor_SMD:CP_Elec_8x10, B.Cu at (173.6, 114.0)
- added C7: 1uF, Capacitor_SMD:C_0805_2012Metric_Pad1.18x1.45mm_HandSolder, F.Cu at (128.6, 125.5)
- added C8: 10nF, Capacitor_SMD:C_0603_1608Metric_Pad1.08x0.95mm_HandSolder, F.Cu at (130.5, 125.5)
- added C9: 1uF, Capacitor_SMD:C_0805_2012Metric_Pad1.18x1.45mm_HandSolder, F.Cu at (144.8, 113.2)
- added IC1: A4954ELPTR-T, Package_SO:TSSOP-16-1EP_4.4x5mm_P0.65mm_EP3x3mm, F.Cu at (124.5, 124.0)
- added J1: Conn_01x02, Connector_PinSocket_2.54mm:PinSocket_1x02_P2.54mm_Horizontal, B.Cu at (149.4, 110.6)
- added J2: SPI, Connector_IDC:IDC-Header_2x05_P2.54mm_Vertical, B.Cu at (136.2, 100.1)
- added J3: SPI_PWR, Connector_PinSocket_2.54mm:PinSocket_1x02_P2.54mm_Vertical, B.Cu at (149.8, 105.8)
- added J4: Conn_01x04, Connector_PinSocket_2.54mm:PinSocket_1x04_P2.54mm_Horizontal, B.Cu at (128.6, 130.4)
- added J5: Conn_01x02, TerminalBlock:TerminalBlock_bornier-2_P5.08mm, B.Cu at (148.1, 118.2)
- added JP1: , Jumper:SolderJumper-2_P1.3mm_Open_Pad1.0x1.5mm, F.Cu at (125.8, 110.1)
- added JP2: , Jumper:SolderJumper-2_P1.3mm_Open_Pad1.0x1.5mm, F.Cu at (128.4, 110.0)
- added JP3: , Jumper:SolderJumper-2_P1.3mm_Open_Pad1.0x1.5mm, F.Cu at (133.7, 105.5)
- added JP4: , Jumper:SolderJumper-2_P1.3mm_Open_Pad1.0x1.5mm, F.Cu at (130.2, 105.5)
- added JP5: , Jumper:SolderJumper-2_P1.3mm_Open_Pad1.0x1.5mm, F.Cu at (146.0, 108.6)
- added JP6: , Jumper:SolderJumper-2_P1.3mm_Open_Pad1.0x1.5mm, F.Cu at (156.3, 125.2)
- added R1: 0.15R, Resistor_SMD:R_0805_2012Metric_Pad1.20x1.40mm_HandSolder, F.Cu at (121.8, 133.2)
- added R2: 0.15R, Resistor_SMD:R_0805_2012Metric_Pad1.20x1.40mm_HandSolder, F.Cu at (129.3, 133.2)
- added R3: 0, Resistor_SMD:R_0805_2012Metric_Pad1.20x1.40mm_HandSolder, F.Cu at (138.1, 114.7)
- added R4: 0, Resistor_SMD:R_0805_2012Metric_Pad1.20x1.40mm_HandSolder, F.Cu at (119.9, 112.3)
- added U1: ATtiny24-20MU, Package_DFN_QFN:QFN-20-1EP_4x4mm_P0.5mm_EP2.6x2.6mm, F.Cu at (117.7, 108.6)
- added U2: AS5047D, Package_SO:TSSOP-14_4.4x5mm_P0.65mm, F.Cu at (131.1, 114.7)
- added U3: TLV70033_SOT353, Package_TO_SOT_SMD:SOT-353_SC-70-5, F.Cu at (142.2, 113.2)
Routing:
- net GND2: track 0.00 -> 130.9 mm
- net GNDREF: track 0.00 -> 79.5 mm
- net MOSI: track 0.00 -> 33.0 mm
- net VD: track 0.00 -> 28.0 mm
- net SCK: track 0.00 -> 27.0 mm
- net VREF1: track 0.00 -> 17.0 mm
- net EXT_CSn: track 0.00 -> 17.0 mm
- net Net-(J2-Pad2): track 0.00 -> 14.6 mm
- net at24CSn2: track 0.00 -> 13.6 mm, vias 0 -> 2
- net MISO: track 0.00 -> 13.3 mm
- net VREF2: track 0.00 -> 13.1 mm
- net Net-(C5-Pad1): track 0.00 -> 13.1 mm
- net +3V3: track 0.00 -> 12.2 mm
- net IN4: track 0.00 -> 11.9 mm, vias 0 -> 2
- net at24CSn: track 0.00 -> 11.8 mm, vias 0 -> 1
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Other:
- outline, holes or cut-outs redrawn

Commit message: Add new updates to driver sch / layout
Parts:
- removed R4: 0, Resistor_SMD:R_0805_2012Metric_Pad1.20x1.40mm_HandSolder
- removed REF** (x4): MountingHole_3.2mm_M3, MountingHole:MountingHole_3.2mm_M3
- U1: footprint Package_DFN_QFN:QFN-20-1EP_4x4mm_P0.5mm_EP2.6x2.6mm -> Package_SO:SOIC-14_3.9x8.7mm_P1.27mm
- moved C6 35.3 mm to (139.7, 124.0), turned to 180 degrees
- moved JP6 23.6 mm to (133.0, 121.5), turned to 0 degrees
- moved C4 7.54 mm to (127.5, 119.0)
- moved C3 6.36 mm to (117.3, 120.7), turned to -90 degrees
- moved C1 4.40 mm to (112.3, 113.3)
- moved U1 0.41 mm to (117.2, 108.5), turned to 180 degrees
- moved R3 0.14 mm to (137.9, 114.5)
Connections:
- U1 pad 1: SCK -> +3V3
- U1 pad 10: unconnected-(U1-Pad10) -> IN1
- U1 pad 11: at24CSn -> IN2
- U1 pad 12: at24CSn2 -> IN3
- U1 pad 13: Reset -> IN4
- U1 pad 14: Net-(U1-Pad14) -> GNDREF
- U1 pad 2: IN1 -> at24CSn
- U1 pad 3: IN2 -> at24CSn2
- U1 pad 4: IN3 -> Reset
- U1 pad 5: IN4 -> VREF2
- U1 pad 6: unconnected-(U1-Pad6) -> VREF1
- U1 pad 7: unconnected-(U1-Pad7) -> MOSI
- U1 pad 8: GNDREF -> MISO
- U1 pad 9: +3V3 -> SCK
Routing:
- net VREF1: track 17.0 -> 44.5 mm, vias 0 -> 2
- net GNDREF: track 79.5 -> 103.4 mm
- net MISO: track 13.3 -> 31.0 mm, vias 0 -> 2
- net Reset: track 10.2 -> 27.6 mm
- net IN1: track 7.80 -> 20.4 mm, vias 2 -> 1
- net SCK: track 27.0 -> 38.7 mm
- net GND2: track 130.9 -> 121.6 mm, vias 0 -> 1
- net IN2: track 7.84 -> 16.8 mm, vias 2 -> 1
- net +3V3: track 12.2 -> 19.9 mm, vias 0 -> 2
- net VREF2: track 13.1 -> 20.5 mm
- net IN3: track 9.25 -> 15.2 mm, vias 2 -> 1
- net MOSI: track 33.0 -> 37.8 mm
- net VD: track 28.0 -> 32.4 mm, vias 0 -> 1
- net IN4: track 11.9 -> 15.7 mm, vias 2 -> 1
- net Net-(U1-Pad14): track 2.09 -> 0.00 mm
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
Commit message: First prototype
Parts:
- added REF**: MountingHole_3.2mm_M3_DIN965, MountingHole:MountingHole_3.2mm_M3_DIN965, F.Cu at (146.5, 99.2)
- added REF**: MountingHole_3.2mm_M3_DIN965, MountingHole:MountingHole_3.2mm_M3_DIN965, F.Cu at (115.5, 99.2)
- added REF**: MountingHole_3.2mm_M3_DIN965, MountingHole:MountingHole_3.2mm_M3_DIN965, F.Cu at (115.7, 130.2)
- added REF**: MountingHole_3.2mm_M3_DIN965, MountingHole:MountingHole_3.2mm_M3_DIN965, F.Cu at (146.6, 130.1)
- moved R1 1.84 mm to (120.1, 132.6)
- moved R2 0.63 mm to (129.5, 132.7)
Connections:
- J2 pad 7: SCK -> Reset
- U1 pad 9: SCK -> Reset
- U2 pad 2: SCK -> Reset
Routing:
- net SCK: track 38.7 -> 0.00 mm
- net +3V3: track 19.9 -> 52.1 mm, vias 2 -> 3
- net VD: track 32.4 -> 58.1 mm
- net Reset: track 27.6 -> 52.5 mm
- net VREF1: track 44.5 -> 61.9 mm
- net VCC: track 10.4 -> 20.0 mm
- net GNDREF: track 103.4 -> 112.9 mm
- net MISO: track 31.0 -> 33.2 mm
- net GND2: track 121.6 -> 123.6 mm

Commit message: AD PCB files
Parts:
- moved REF** 0.16 mm to (115.5, 130.2)
- moved REF** 0.11 mm to (146.5, 130.2)
